Commit message: added robot state publisher, rviz

File: snu_sdx_controller/dyros_robot_controller/husky_controller/robot/husky.urdf (robot description, URDF)
Before this commit: robot husky, 8 links, 7 joints
Links:
- added link front_bumper_link; visual mesh filename=package://husky_description/meshes/bumper.dae
- added link rear_bumper_link; visual mesh filename=package://husky_description/meshes/bumper.dae
- added link top_chassis_link; visual mesh filename=package://husky_description/meshes/top_chassis.dae
- added link top_plate_front_link
- added link top_plate_link; collision mesh filename=package://husky_description/meshes/top_plate.stl; visual mesh filename=package://husky_description/meshes/top_plate.dae
- added link top_plate_rear_link
- added link user_rail_link; visual mesh filename=package://husky_description/meshes/user_rail.dae
Joints:
- added joint front_bumper: type fixed, parent base_link, child front_bumper_link, origin xyz=0.48 0 0.091 rpy=0 0 0
- added joint rear_bumper: type fixed, parent base_link, child rear_bumper_link, origin xyz=-0.48 0 0.091 rpy=0 0 3.141592
- added joint top_chassis_joint: type fixed, parent base_link, child top_chassis_link
- added joint top_plate_front_joint: type fixed, parent top_plate_link, child top_plate_front_link, origin xyz=0.36367 0 0.00639 rpy=0 0 0
- added joint top_plate_joint: type fixed, parent base_link, child top_plate_link, origin xyz=0.0812 0 0.245 rpy=0 0 0
- added joint top_plate_rear_joint: type fixed, parent top_plate_link, child top_plate_rear_link, origin xyz=-0.36633 0 0.00639 rpy=0 0 0
- added joint user_rail: type fixed, parent base_link, child user_rail_link, origin xyz=0.272 0 0.245 rpy=0 0 0
