Commit message: Added MOB, compensating f/t sensor bias

File: snu_sdx_controller/dyros_robot_controller/fr3_husky_controller/robot/fr3.urdf (robot description, URDF)
Before this commit: robot fr3, 10 links, 9 joints
Links:
- link fr3_link8: mass None -> 0.73

File: snu_sdx_controller/dyros_robot_controller/fr3_husky_controller/robot/fr3_husky.urdf (robot description, URDF)
Before this commit: robot fr3_husky, 21 links, 20 joints
Links:
- removed link fr3_hand
- removed link fr3_leftfinger
- removed link fr3_rightfinger
- removed link hand_tcp
- added link front_bumper_link; visual mesh filename=package://husky_description/meshes/bumper.dae
- added link rear_bumper_link; visual mesh filename=package://husky_description/meshes/bumper.dae
- added link top_chassis_link; visual mesh filename=package://husky_description/meshes/top_chassis.dae
- added link top_plate_front_link
- added link top_plate_link; collision mesh filename=package://husky_description/meshes/roas_dyros.STL; visual mesh filename=package://husky_description/meshes/roas_dyros.STL
- added link top_plate_rear_link
- added link user_rail_link; visual mesh filename=package://husky_description/meshes/user_rail.dae
- link fr3_link8: mass None -> 0.73
Joints:
- removed joint fr3_finger_joint1
- removed joint fr3_finger_joint2
- removed joint fr3_hand_joint
- removed joint fr3_mani_joint1
- removed joint fr3_mani_joint2
- removed joint fr3_mani_joint3
- removed joint fr3_mani_joint4
- removed joint fr3_mani_joint5
- removed joint fr3_mani_joint6
- removed joint fr3_mani_joint7
- removed joint fr3_mani_joint8
- removed joint hand_tcp_joint
- added joint fr3_joint1: type revolute, parent fr3_link0, child fr3_link1, origin xyz=0 0 0.333 rpy=0 0 0, axis 0 0 1, limit lower=-2.7437 upper=2.7437 effort=87.0 velocity=2.62
- added joint fr3_joint2: type revolute, parent fr3_link1, child fr3_link2, origin xyz=0 0 0 rpy=-1.570796326794897 0 0, axis 0 0 1, limit lower=-1.7837 upper=1.7837 effort=87.0 velocity=2.62
- added joint fr3_joint3: type revolute, parent fr3_link2, child fr3_link3, origin xyz=0 -0.316 0 rpy=1.570796326794897 0 0, axis 0 0 1, limit lower=-2.9007 upper=2.9007 effort=87.0 velocity=2.62
- added joint fr3_joint4: type revolute, parent fr3_link3, child fr3_link4, origin xyz=0.0825 0 0 rpy=1.570796326794897 0 0, axis 0 0 1, limit lower=-3.0421 upper=-0.1518 effort=87.0 velocity=2.62
- added joint fr3_joint5: type revolute, parent fr3_link4, child fr3_link5, origin xyz=-0.0825 0.384 0 rpy=-1.570796326794897 0 0, axis 0 0 1, limit lower=-2.8065 upper=2.8065 effort=12.0 velocity=5.26
- added joint fr3_joint6: type revolute, parent fr3_link5, child fr3_link6, origin xyz=0 0 0 rpy=1.570796326794897 0 0, axis 0 0 1, limit lower=0.5445 upper=4.5169 effort=12.0 velocity=4.18
- added joint fr3_joint7: type revolute, parent fr3_link6, child fr3_link7, origin xyz=0.088 0 0 rpy=1.570796326794897 0 0, axis 0 0 1, limit lower=-3.0159 upper=3.0159 effort=12.0 velocity=5.26
- added joint fr3_joint8: type fixed, parent fr3_link7, child fr3_link8, origin xyz=0 0 0.107 rpy=0 0 0
- added joint front_bumper: type fixed, parent base_link, child front_bumper_link, origin xyz=0.48 0 0.091 rpy=0 0 0
- added joint rear_bumper: type fixed, parent base_link, child rear_bumper_link, origin xyz=-0.48 0 0.091 rpy=0 0 3.141592
- added joint top_chassis_joint: type fixed, parent base_link, child top_chassis_link
- added joint top_plate_front_joint: type fixed, parent top_plate_link, child top_plate_front_link, origin xyz=0.36367 0 0.00639 rpy=0 0 0
- added joint top_plate_joint: type fixed, parent base_link, child top_plate_link, origin xyz=0 0 0 rpy=0 0 0
- added joint top_plate_rear_joint: type fixed, parent top_plate_link, child top_plate_rear_link, origin xyz=-0.36633 0 0.00639 rpy=0 0 0
- added joint user_rail: type fixed, parent base_link, child user_rail_link, origin xyz=0.272 0 0.245 rpy=0 0 0
- joint fr3_base_joint: origin xyz=0.36 0 0.25 rpy=0 0 0 -> xyz=0.335 0 0.255 rpy=0 0 0
